Commit message: new design

File: src/aeriaman/urdf/man.xacro (robot description, xacro)
@@ -26,7 +26,7 @@
 <!-- Base Link -->
 <link name="base_link">
-<visual> <origin xyz="0 0 0.1" rpy="0 0 0" /> <geometry> <box size= "2 2 0.2" /> <material name="blue"> <color rgba="0 0 .8 1"/> </material></geometry> </visual>
-<collision> <origin xyz="0 0 0.1" rpy="0 0 0" /> <geometry> <box size= "2 2 0.2" /> </geometry> </collision>
-<inertial> <origin xyz="0 0 0.1" rpy="0 0 0" /> <mass value="${mass1}" /> <inertia ixx="${mass1 / 12.0 * (2*2 + 0.2*0.2)}" ixy="0.0" ixz="0.0"
+<visual> <origin xyz="0 0 2" rpy="0 0 0" /> <geometry> <box size= "2 2 0.2" /> <material name="blue"> <color rgba="0 0 .8 1"/> </material></geometry> </visual>
+<collision> <origin xyz="0 0 2" rpy="0 0 0" /> <geometry> <box size= "2 2 0.2" /> </geometry> </collision>
+<inertial> <origin xyz="0 0 2" rpy="0 0 0" /> <mass value="${mass1}" /> <inertia ixx="${mass1 / 12.0 * (2*2 + 0.2*0.2)}" ixy="0.0" ixz="0.0"
 iyy="${mass1 / 12.0 * (0.2*0.2 + 2*2)}" iyz="0.0"
 izz="${mass1 / 12.0 * (2*2 + 2*2)}"/> </inertial>
@@ -36,13 +36,13 @@
 <joint name="jf" type="fixed">
 <parent link="base_link" /> <child link="sh_link" />
-<origin xyz="0 ${width} 0.2" rpy="0 0 0" />
+<origin xyz="0 ${width} -0.1" rpy="0 0 0" />
 <axis xyz="0 0 0" /> <dynamics damping="${damp}" />
 <limit effort="0" velocity="0" lower="0" upper="0" /> </joint>
-<!-- done== origin from the last link size-->
+<!-- done== origin from the last link size l1zorigin-l1zsize+l2zsize/2-->
 <!-- Link -->
 <link name="sh_link">
-<visual> <origin xyz="0 0 0.05" rpy="0 0 0" /> <geometry> <box size= "0.1 0.1 0.1" /> <material name="blue"> <color rgba="0 0 .8 1"/> </material></geometry> </visual>
-<collision> <origin xyz="0 0 0.05" rpy="0 0 0" /> <geometry> <box size= "0.1 0.1 0.1" /> </geometry> </collision>
-<inertial> <origin xyz="0 0 0.05" rpy="0 0 0" /> <mass value="${mass2}" />
+<visual> <origin xyz="0 0 1.95" rpy="0 0 0" /> <geometry> <box size= "0.1 0.1 0.1" /> <material name="blue"> <color rgba="0 0 .8 1"/> </material></geometry> </visual>
+<collision> <origin xyz="0 0 1.95" rpy="0 0 0" /> <geometry> <box size= "0.1 0.1 0.1" /> </geometry> </collision>
+<inertial> <origin xyz="0 0 1.95" rpy="0 0 0" /> <mass value="${mass2}" />
 <inertia ixx="${mass2 / 12.0 * (0.1*0.1 + 0.1*0.1)}" ixy="0.0" ixz="0.0"
 iyy="${mass2 / 12.0 * (0.1*0.1 + 0.1*0.1)}" iyz="0.0"
@@ -52,5 +52,5 @@
 <joint name="j1" type="revolute">
 <parent link="sh_link" /> <child link="arm_shlink" />
-<origin xyz="0 0 0.1" rpy="0 0 0" />
+<origin xyz="0 0 1.9" rpy="0 0 0" />
 <axis xyz="0 1 0"/> <dynamics damping="${damp}" />
 <limit effort="1000.0" velocity="0.5" lower="-1.5" upper="1.5" />
@@ -58,7 +58,7 @@
 <!-- Link -->
 <link name="arm_shlink">
-<visual> <origin xyz="0 0 0.1" rpy="0 0 0" /> <geometry> <box size= "0.1 0.1 0.2" /> <material name="blue"> <color rgba="0 0 .8 1"/> </material></geometry> </visual>
-<collision> <origin xyz="0 0 0.1" rpy="0 0 0" /> <geometry> <box size= "0.1 0.1 0.2" /> </geometry> </collision>
-<inertial> <origin xyz="0 0 0.1" rpy="0 0 0" /> <mass value="${mass3}" /> <inertia
+<visual> <origin xyz="0 0 -0.1" rpy="0 0 0" /> <geometry> <box size= "0.1 0.1 0.2" /> <material name="blue"> <color rgba="0 0 .8 1"/> </material></geometry> </visual>
+<collision> <origin xyz="0 0 -0.1" rpy="0 0 0" /> <geometry> <box size= "0.1 0.1 0.2" /> </geometry> </collision>
+<inertial> <origin xyz="0 0 -0.1" rpy="0 0 0" /> <mass value="${mass3}" /> <inertia
 ixx="${mass3 / 12.0 * (0.1*0.1 + 0.2*0.2)}" ixy="0.0" ixz="0.0"
 iyy="${mass3 / 12.0 * (0.2*0.2 + 0.1*0.1)}" iyz="0.0"
@@ -69,5 +69,5 @@
 <joint name="j2" type="revolute">
 <parent link="arm_shlink" /> <child link="forearm_link" />
-<origin xyz="0 0 0.2" rpy="0 0 0" />
+<origin xyz="0 0 -0.2" rpy="0 0 0" />
 <axis xyz="1 0 0" /> <dynamics damping="${damp}" />
 <limit effort="1000.0" velocity="0.5" lower="-1.5" upper="1.5" /> </joint>
@@ -75,7 +75,7 @@
 <!-- Link -->
 <link name="forearm_link">
-<visual> <origin xyz="0 0 0.5" rpy="0 0 0" /> <geometry> <box size= "0.1 0.1 1" /> <material name="blue"> <color rgba="0 0 .8 1"/> </material></geometry> </visual>
-<collision> <origin xyz="0 0 0.5" rpy="0 0 0" /> <geometry> <box size= "0.1 0.1 1" /> </geometry> </collision>
-<inertial> <origin xyz="0 0 0.5" rpy="0 0 0" /> <mass value="${mass4}" /> <inertia
+<visual> <origin xyz="0 0 -0.5" rpy="0 0 0" /> <geometry> <box size= "0.1 0.1 1" /> <material name="blue"> <color rgba="0 0 .8 1"/> </material></geometry> </visual>
+<collision> <origin xyz="0 0 -0.5" rpy="0 0 0" /> <geometry> <box size= "0.1 0.1 1" /> </geometry> </collision>
+<inertial> <origin xyz="0 0 -0.5" rpy="0 0 0" /> <mass value="${mass4}" /> <inertia
 ixx="${mass4 / 12.0 * (0.1*0.1 + 1)}" ixy="0.0" ixz="0.0"
 iyy="${mass4 / 12.0 * (1 + 0.1*0.1)}" iyz="0.0"
@@ -86,5 +86,5 @@
 <joint name="j3" type="revolute">
 <parent link="forearm_link" /> <child link="arm_link" />
-<origin xyz="0 0 1" rpy="0 0 0" />
+<origin xyz="0 0 -1" rpy="0 0 0" />
 <axis xyz="1 0 0" /> <dynamics damping="${damp}" />
 <limit effort="1000.0" velocity="0.5" lower="-1.5" upper="1.5" /> </joint>
@@ -92,7 +92,55 @@
 <!-- Link -->
 <link name="arm_link">
-<visual> <origin xyz="0 0 0.4" rpy="0 0 0" /> <geometry> <box size= "0.1 0.1 0.8" /> <material name="blue"> <color rgba="0 0 .8 1"/> </material></geometry> </visual>
-<collision> <origin xyz="0 0 0.4" rpy="0 0 0" /> <geometry> <box size= "0.1 0.1 0.8" /> </geometry> </collision>
-<inertial> <origin xyz="0 0 0.4" rpy="0 0 0" /> <mass value="${mass5}" /> <inertia ixx="${mass5 / 12.0 * (0.1*0.1 + 0.8*0.8)}" ixy="0.0" ixz="0.0"
+<visual> <origin xyz="0 0 -0.4" rpy="0 0 0" /> <geometry> <box size= "0.1 0.1 0.8" /> <material name="blue"> <color rgba="0 0 .8 1"/> </material></geometry> </visual>
+<collision> <origin xyz="0 0 -0.4" rpy="0 0 0" /> <geometry> <box size= "0.1 0.1 0.8" /> </geometry> </collision>
+<inertial> <origin xyz="0 0 -0.4" rpy="0 0 0" /> <mass value="${mass5}" /> <inertia ixx="${mass5 / 12.0 * (0.1*0.1 + 0.8*0.8)}" ixy="0.0" ixz="0.0"
+iyy="${mass5 / 12.0 * (0.8*0.8 + 0.1*0.1)}" iyz="0.0"
+izz="${mass5 / 12.0 * (0.1*0.1 + 0.1*0.1)}"/> </inertial>
+</link>
+<!-- done link== origin from the center of gravity-->
+<!-- Joint -->
+<joint name="j4" type="revolute">
+<parent link="arm_link" /> <child link="hand_1_link" />
+<origin xyz="0 0 -0.8" rpy="0 0 0" />
+<axis xyz="0 0 1" /> <dynamics damping="${damp}" />
+<limit effort="1000.0" velocity="0.5" lower="-1.5" upper="1.5" /> </joint>
+<!-- done joint== origin from the last link's size-->
+<!-- Link -->
+<link name="hand_1_link">
+<visual> <origin xyz="0 0 -0.05" rpy="0 0 0" /> <geometry> <box size= "0.1 0.1 0.1" /> <material name="blue"> <color rgba="0 0 .8 1"/> </material></geometry> </visual>
+<collision> <origin xyz="0 0 -0.05" rpy="0 0 0" /> <geometry> <box size= "0.1 0.1 0.8" /> </geometry> </collision>
+<inertial> <origin xyz="0 0 -0.05" rpy="0 0 0" /> <mass value="${mass5}" /> <inertia ixx="${mass5 / 12.0 * (0.1*0.1 + 0.8*0.8)}" ixy="0.0" ixz="0.0"
+iyy="${mass5 / 12.0 * (0.8*0.8 + 0.1*0.1)}" iyz="0.0"
+izz="${mass5 / 12.0 * (0.1*0.1 + 0.1*0.1)}"/> </inertial>
+</link>
+<!-- done link== origin from the center of gravity-->
+<!-- Joint -->
+<joint name="j5" type="revolute">
+<parent link="hand_1_link" /> <child link="hand_2_link" />
+<origin xyz="0 0 -0.1" rpy="0 0 0" />
+<axis xyz="1 0 0" /> <dynamics damping="${damp}" />
+<limit effort="1000.0" velocity="0.5" lower="-1.5" upper="1.5" /> </joint>
+<!-- done joint== origin from the last link's size-->
+<!-- Link -->
+<link name="hand_2_link">
+<visual> <origin xyz="0 0 -0.05" rpy="0 0 0" /> <geometry> <box size= "0.1 0.1 0.1" /> <material name="blue"> <color rgba="0 0 .8 1"/> </material></geometry> </visual>
+<collision> <origin xyz="0 0 -0.05" rpy="0 0 0" /> <geometry> <box size= "0.1 0.1 0.8" /> </geometry> </collision>
+<inertial> <origin xyz="0 0 -0.05" rpy="0 0 0" /> <mass value="${mass5}" /> <inertia ixx="${mass5 / 12.0 * (0.1*0.1 + 0.8*0.8)}" ixy="0.0" ixz="0.0"
+iyy="${mass5 / 12.0 * (0.8*0.8 + 0.1*0.1)}" iyz="0.0"
+izz="${mass5 / 12.0 * (0.1*0.1 + 0.1*0.1)}"/> </inertial>
+</link>
+<!-- done link== origin from the center of gravity-->
+<!-- Joint -->
+<joint name="j6" type="revolute">
+<parent link="hand_2_link" /> <child link="hand_3_link" />
+<origin xyz="0 0 -0.1" rpy="0 0 0" />
+<axis xyz="0 1 0" /> <dynamics damping="${damp}" />
+<limit effort="1000.0" velocity="0.5" lower="-1.5" upper="1.5" /> </joint>
+<!-- done joint== origin from the last link's size-->
+<!-- Link -->
+<link name="hand_3_link">
+<visual> <origin xyz="0 0 -0.2" rpy="0 0 0" /> <geometry> <box size= "0.4 0.1 0.4" /> <material name="blue"> <color rgba="0 0 .8 1"/> </material></geometry> </visual>
+<collision> <origin xyz="0 0 -0.05" rpy="0 0 0" /> <geometry> <box size= "0.1 0.1 0.8" /> </geometry> </collision>
+<inertial> <origin xyz="0 0 -0.05" rpy="0 0 0" /> <mass value="${mass5}" /> <inertia ixx="${mass5 / 12.0 * (0.1*0.1 + 0.8*0.8)}" ixy="0.0" ixz="0.0"
 iyy="${mass5 / 12.0 * (0.8*0.8 + 0.1*0.1)}" iyz="0.0"
 izz="${mass5 / 12.0 * (0.1*0.1 + 0.1*0.1)}"/> </inertial>

Commit message: fix ros_control

File: src/aeriaman/urdf/man.xacro (robot description, xacro)
@@ -176,3 +176,33 @@
     </actuator>
 </transmission>
+<transmission name="t4">
+    <type>transmission_interface/SimpleTransmission</type>
+    <joint name="j4">
+      <hardwareInterface>hardware_interface/EffortJointInterface</hardwareInterface>
+    </joint>
+    <actuator name="m4">
+      <hardwareInterface>hardware_interface/EffortJointInterface</hardwareInterface>
+      <mechanicalReduction>1</mechanicalReduction>
+    </actuator>
+</transmission>
+<transmission name="t5">
+    <type>transmission_interface/SimpleTransmission</type>
+    <joint name="j5">
+      <hardwareInterface>hardware_interface/EffortJointInterface</hardwareInterface>
+    </joint>
+    <actuator name="m5">
+      <hardwareInterface>hardware_interface/EffortJointInterface</hardwareInterface>
+      <mechanicalReduction>1</mechanicalReduction>
+    </actuator>
+</transmission>
+<transmission name="t6">
+    <type>transmission_interface/SimpleTransmission</type>
+    <joint name="j6">
+      <hardwareInterface>hardware_interface/EffortJointInterface</hardwareInterface>
+    </joint>
+    <actuator name="m6">
+      <hardwareInterface>hardware_interface/EffortJointInterface</hardwareInterface>
+      <mechanicalReduction>1</mechanicalReduction>
+    </actuator>
+</transmission>
 </robot>
